Commit message: 3D Point Cloud + Gazebo GUI

File: src/xarm_description/urdf/xarm6_with_gripper.urdf (robot description, URDF)
Before this commit: robot xarm6_with_gripper, 15 links, 14 joints
Links:
- added link camera_bottom_screw_frame, mass 0.00583601107155577; visual mesh filename=package://orbbec_description/meshes/astra2/camera_bottom_sc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
- added link camera_color_frame, mass 7.68929599151334E-05; visual mesh filename=package://orbbec_description/meshes/astra2/camera_colorl_fr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
- added link camera_color_optical_frame
- added link camera_depth_frame, mass 0.000608348661221201; visual mesh filename=package://orbbec_description/meshes/astra2/camera_depth_fra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
- added link camera_depth_optical_frame
- added link camera_ir_frame
- added link camera_ir_optical_frame
- added link camera_link, mass 0.0101524380243699; visual mesh filename=package://orbbec_description/meshes/astra2/base_link.STL
Joints:
- added joint camera_bottom_screw_joint: type fixed, parent camera_link, child camera_bottom_screw_frame, origin xyz=-0.012323995999904 -0.0374999999985815 -0.0281503197112 rpy=0 0 0
- added joint camera_color_joint: type fixed, parent camera_depth_frame, child camera_color_frame, origin xyz=0.0025420000310987234 -0.01850000023841858 0 rpy=0 0 0
- added joint camera_color_optical_joint: type fixed, parent camera_color_frame, child camera_color_optical_frame, origin xyz=0 0 0 rpy=-1.5707963267949 0 -1.5707963267949
- added joint camera_depth_joint: type fixed, parent camera_link, child camera_depth_frame, origin xyz=0 0 0 rpy=0 0 0
- added joint camera_depth_optical_joint: type fixed, parent camera_depth_frame, child camera_depth_optical_frame, origin xyz=0 0 0 rpy=-1.5707963267949 0 -1.5707963267949
- added joint camera_ir_joint: type fixed, parent camera_depth_frame, child camera_ir_frame, origin xyz=0 0 0 rpy=0 0 0
- added joint camera_ir_optical_joint: type fixed, parent camera_ir_frame, child camera_ir_optical_frame, origin xyz=0 0 0 rpy=-1.5707963267949 0 -1.5707963267949
- added joint camera_mount_joint: type fixed, parent world, child camera_link, origin xyz=1.0 0.0 0.6 rpy=0 0.45 3.14159
